File: hardware/pcb/StarShield/power/power.kicad_sch (KiCad schematic)
At the start: 18 parts, among them J1 USB_C_Receptacle_USB2.0_16P, J2 B2B-PH-K-S, Q1 AO3401A, Q2 2N7002, U1 BQ24072RGT

Commit message: feat(power): 按社区成熟方案落地五处改动（VBUS 保险丝 / R_ILIM 1.5k / 补装 R_TMR / EP 热过孔 / C 倍率换算）
1) 新增 F1 = 500mA 保险丝装在 VBUS 侧（VBUS->F1->VCHG_IN->U1.IN），照抄 nightliner 的位置。不可照抄 Conejo：它那颗串在电池路径上，而 RGB 全部放电电流都走那条路 => 必然误断。VCHG_IN 含 U1.IN(power_in) 故需 PWR_FLAG。

2) R_ILIM 1.6k -> 1.5k（osprey/designguide 值）。3) 补装 R_TMR = 47k，TMR 不再悬空 —— 修正本项目原先的错误结论：内部默认只有 5h，而 ICHG 0.5A x 3000mAh 仅 CC 段就约 6.2h，悬空会在充满前被安全定时器掐断；原先用定时器节流变慢论证够用是错的。

4) U1 封装改为 VQFN-16-1EP_3x3mm_P0.5mm_EP1.6x1.6mm_ThermalVias（nightliner 同做法）。5) R_ISET 保持 1.78k 不照抄社区的 3.9k —— 关键发现：社区 0.23A 是给 200-500mAh 电芯的 0.46-0.91C，照抄到 3000mAh 会变成 0.077C（约13h）；R_ISET 要按 C 倍率换算而非绝对电流。

修掉新坑：给局部网络挂全局标签接 PWR_FLAG 会触发 ERC [same_local_global_label]，PWR_FLAG 的标签类别必须与网络本身一致。

验收：20 元件 / 72 条引脚连接；verify_power 全过（新增保险丝与 TMR 具名断言、NC 数 8->7）；四校验器全绿；两轮生成器哈希一致；ERC 0 error / 2 warning。新增待决策 P15（保险丝降额复核）。
Parts:
- added F1: 500mA, Fuse:Fuse_0603_1608Metric, symbol Device:Fuse
- added R10: 47k, Resistor_SMD:R_0603_1608Metric, symbol Device:R
- R3: value 1.6k -> 1.5k; Note USB500 档下不参与限流，但必须装（悬空=关闭充电） -> USB500 档下不参与限流，但必须装（悬空=关闭充电）；取值同社区 1.5k
- R4: Note ICHG=890/1.78k≈0.5A，1% -> ICHG=890/1.78k≈0.5A=0.17C@3000mAh，1%
- U1: footprint Package_DFN_QFN:VQFN-16-1EP_3x3mm_P0.5mm_EP1.6x1.6mm -> Package_DFN_QFN:VQFN-16-1EP_3x3mm_P0.5mm_EP1.6x1.6mm_ThermalVias; Note EP(17) 必须焊到接地铜皮 + 热过孔 -> EP(17) 必须焊到接地铜皮；封装已选 ThermalVias 变体（社区同做法）
Connections:
- net GND: now also R10.2
- net VBUS: now also F1.1; no longer C1.1, U1.13 (IN)
- net TMR: now reaches U1.14 (TMR)
- net TMR: now also R10.1
- new net VCHG_IN: C1.1, F1.2, U1.13 (IN)
- no-connect marks 8 -> 7
Other:
- note added: "【取值依据】U1=BQ24072RGT。ICHG = 890 / R_ISET = 0.5 A（=0.17C @3000mAh）；EN2=0 且 EN1=1 选 USB500 档（输入上限 500 mA）；~CE 接 VSS 常开；TD 接 VSS 使能充电终止；TS 经 10k 到 VSS 禁用温度监测；TMR 装 47k（6.25h 安全定时，默认 5h 不够）；VBUS 经 F1（500mA）后进 IN。取值与社区成熟方案对照见 docs/power-architecture.md 3.4"
- note added: "【本版留空 / 未决项】P2 与 P10：USB-C 的 D+ D- SBU 全部 NC（第一版 USB-C 仅充电）；U1 的 ~PGOOD 悬空（预留测试点）。F1 保险丝的额定值待按所选料号的降额曲线复核。详见 docs/power-architecture.md 第 6 节待办"
- note removed: "【取值依据】U1=BQ24072RGT。ICHG = 890 / R_ISET = 0.5 A；EN2=0 且 EN1=1 选 USB500 档（输入上限 500 mA）；~CE 接 VSS 常开；TD 接 VSS 使能充电终止；TS 经 10k 到 VSS 禁用温度监测；TMR 悬空 = 内部默认定时（预充 30 min / 快充 5 h）"
- note removed: "【本版留空 / 未决项】P2 与 P10：USB-C 的 D+ D- SBU 全部 NC（第一版 USB-C 仅充电）；U1 的 ~PGOOD 悬空（预留测试点）；U1 的 TMR 悬空。详见 docs/power-architecture.md 第 6 节待办"

Commit message: feat(power): 电池改为 2x5000mAh 并联（10000mAh），TMR 改接 VSS 禁用安全定时器
【容量】按用户决定，电池由 3000mAh 单节改为 2x5000mAh 并联（1S2P，共用一块 PCM）。串联被电气排除：数据手册 8.1 节 BAT 绝对最大额定仅 -0.3…5V，2S 满电 8.4V 超限 68%。

【对标】新增 research/keyboard-battery-capacity-precedent.md（商用 10000mAh 键盘做法）：AULA F87S 官方承认不是单体 10000mAh 而是 2x5000 并联，理由与我们独立推出的一致（单体太厚），并指出可分置左右两侧平衡配重；Kzzi K98PRO 10000mAh 配 DC5V/1.4A；Hola87 10000mAh 配 DC5V/350mA（需 28.6h）。

【关键发现】消费级充电 IC 普遍没有「最长充电时间」限制 —— Hola87 的 28.6h 反证了这点。BQ24072 的 tMAXCHG 是 TI 的额外高级特性，不是行业必需项；真正的保命线是电芯保护板 + 4.2V 恒压 + 终止电流检测，三者本项目都有。

【改动】R_TMR 移除，TMR 直接接 VSS（数据手册明确支持）。原因：tMAXCHG 上限 = 10 x 72kΩ x 60s/kΩ = 12h（typ 9.6h），而 0.5A 充满 10Ah 需约 20.6h => 任何 R_TMR 都会中途掐断，用户永远只用到约一半容量。这一步同时推翻了同日稍早「必须装 47kΩ」的结论（它建立在 3000mAh 之上）。

【不变】充电电流维持 USB500 档 0.5A。切 ILIM 档虽能约 6.7h 充满，但超 USB-C 声明 2.6-3 倍，且耗散 2W => +87C 必然热调节降流 => 实际仍可能超时，属不确定方案，本项目一贯避免。

【新增约束】power-architecture.md 新增 3.5（对标与三条路线）与 3.6（采购要求）：必须买一体化 1S2P 单 PCM 包（两块各自带保护板的电芯直接并联会互充 + 阈值失配）；PCM 过流阈值须 >2A（RGB 全亮约 1.9A）；引出线 AWG #24、接头 JST-PH；电池仓 6.5x51x84mm -> 约 10.5x110x68mm，机壳深 >=8.5-9mm -> >=11mm。

【同步】容量相关算例更新（ADR-0002/0005/0010、decisions、hardware-geometry G5、bq24072-pinout 3.5）；ADR-0002 加勘误（原文「1.5-2 小时充满」作废）。

【验收】19 元件 / 70 条引脚连接；四校验器全绿；两轮生成器哈希一致；ERC 仍 0 error / 2 warning。
Parts:
- removed R10: 47k, Resistor_SMD:R_0603_1608Metric, symbol Device:R
- J2: Note pin1=电池+ pin2=GND（⚠️ 极性不可反） -> pin1=电池+ pin2=GND（极性不可反）；须接 1S2P 单 PCM 电池包 10000mAh
- R4: Note ICHG=890/1.78k≈0.5A=0.17C@3000mAh，1% -> ICHG=890/1.78k≈0.5A=0.05C@10000mAh，1%
Connections:
- net TMR is gone; now on net GND: U1.14 (TMR)
Other:
- note added: "【取值依据】U1=BQ24072RGT。电池 = 2x5000mAh 并联（1S2P 共用一块 PCM，共 10000mAh）。ICHG = 890 / R_ISET = 0.5 A（=0.05C @10000mAh）；EN2=0 且 EN1=1 选 USB500 档（输入上限 500 mA）；~CE 接 VSS 常开；TD 接 VSS 使能充电终止；TS 经 10k 到 VSS 禁用温度监测；TMR 接 VSS 禁用所有安全定时器（充满 10000mAh 约需 20h，超出定时器 12h 上限）。VBUS 经 F1（500mA）后进 IN。容量与商用键盘对照见 docs/power-architecture.md 3.5"
- note added: "【投板后必须实测】1) AO3401A 在 Vgs 约 -0.9 V 时的关断漏电（标 UNVERIFIED）2) RGB 峰值电流下 OUT 压降是否仍在 250 mV 以内 3) 深睡整机电流（目标约 20 uA）4) TMR 接 VSS 后充电能否正常走到 4.2 V 并靠终止电流判据结束（安全定时器已禁用）"
- note added: "【电池与连接器约束】J2 为 JST-PH 2.0，额定 2 A（限 AWG #24 条件）。RGB 全亮峰值约 2.4 A 超过该额定，pigtail 请指定 AWG #24。电池须为 1S2P 一体化包（两块 5000mAh 共用一块 PCM），不可用两块各自带保护板的电芯直接并联（会互充，且两块保护板阈值失配）；PCM 的过流保护阈值必须大于 2A，否则 RGB 全亮会触发保护断电"
- note removed: "【取值依据】U1=BQ24072RGT。ICHG = 890 / R_ISET = 0.5 A（=0.17C @3000mAh）；EN2=0 且 EN1=1 选 USB500 档（输入上限 500 mA）；~CE 接 VSS 常开；TD 接 VSS 使能充电终止；TS 经 10k 到 VSS 禁用温度监测；TMR 装 47k（6.25h 安全定时，默认 5h 不够）；VBUS 经 F1（500mA）后进 IN。取值与社区成熟方案对照见 docs/power-architecture.md 3.4"
- note removed: "【投板后必须实测】1) AO3401A 在 Vgs 约 -0.9 V 时的关断漏电（标 UNVERIFIED）2) RGB 峰值电流下 OUT 压降是否仍在 250 mV 以内 3) 深睡整机电流（目标约 20 uA）"
- note removed: "【连接器约束】J2 为 JST-PH 2.0，额定 2 A（限 AWG #24 条件）。RGB 全亮峰值约 2.4 A 超过该额定，不可靠接插件承载全亮电流；pigtail 请指定 AWG #24"
Changed lines of the file:
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@@
-		(pin "1")
-	)
-	(wire (pts (xy 95.25 135.89) (xy 95.25 133.35))
-		(stroke (width 0) (type default)))
-	(label "TMR" (at 95.25 133.35 90) (fields_autoplaced yes)
-		(effects (font (size 1.27 1.27)) (justify left bottom))
-	)
-	(wire (pts (xy 95.25 143.51) (xy 95.25 146.05))
-		(stroke (width 0) (type default)))
-	(symbol (lib_id "power:GND") (at 95.25 146.05 0) (unit 1)
-		(exclude_from_sim no) (in_bom yes) (on_board yes) (dnp no) (fields_autoplaced yes)
-		(property "Reference" "#PWR0189" (at 95.25 140.97 0)
-			(effects (font (size 1.27 1.27)) (hide yes)))
-		(property "Value" "GND" (at 95.25 151.13 0)
-			(effects (font (size 1.27 1.27)) (hide yes)))
-		(property "Footprint" "" (at 95.25 146.05 0)
-			(effects (font (size 1.27 1.27)) (hide yes)))
-		(property "Datasheet" "" (at 95.25 146.05 0)
-			(effects (font (size 1.27 1.27)) (hide yes)))
 		(pin "1")
 	)
@@
 	(symbol (lib_id "power:GND") (at 137.16 91.44 270) (unit 1)
 		(exclude_from_sim no) (in_bom yes) (on_board yes) (dnp no) (fields_autoplaced yes)
-		(property "Reference" "#PWR0188" (at 137.16 86.36 0)
+		(property "Reference" "#PWR0189" (at 137.16 86.36 0)
 			(effects (font (size 1.27 1.27)) (hide yes)))
 		(property "Value" "GND" (at 137.16 96.52 0)
@@
 	(symbol (lib_id "power:GND") (at 137.16 99.06 270) (unit 1)
 		(exclude_from_sim no) (in_bom yes) (on_board yes) (dnp no) (fields_autoplaced yes)
-		(property "Reference" "#PWR0187" (at 137.16 93.98 0)
+		(property "Reference" "#PWR0188" (at 137.16 93.98 0)
 			(effects (font (size 1.27 1.27)) (hide yes)))
 		(property "Value" "GND" (at 137.16 104.14 0)
@@
 	(symbol (lib_id "power:GND") (at 152.4 114.3 0) (unit 1)
 		(exclude_from_sim no) (in_bom yes) (on_board yes) (dnp no) (fields_autoplaced yes)
-		(property "Reference" "#PWR0186" (at 152.4 109.22 0)
+		(property "Reference" "#PWR0187" (at 152.4 109.22 0)
 			(effects (font (size 1.27 1.27)) (hide yes)))
 		(property "Value" "GND" (at 152.4 119.38 0)
@@
 	(wire (pts (xy 139.7 93.98) (xy 137.16 93.98))
 		(stroke (width 0) (type default)))
-	(label "TMR" (at 137.16 93.98 180) (fields_autoplaced yes)
-		(effects (font (size 1.27 1.27)) (justify right bottom))
+	(symbol (lib_id "power:GND") (at 137.16 93.98 270) (unit 1)
+		(exclude_from_sim no) (in_bom yes) (on_board yes) (dnp no) (fields_autoplaced yes)
+		(property "Reference" "#PWR0186" (at 137.16 88.9 0)
+			(effects (font (size 1.27 1.27)) (hide yes)))
+		(property "Value" "GND" (at 137.16 99.06 0)
+			(effects (font (size 1.27 1.27)) (hide yes)))
+		(property "Footprint" "" (at 137.16 93.98 0)
+			(effects (font (size 1.27 1.27)) (hide yes)))
+		(property "Datasheet" "" (at 137.16 93.98 0)
+			(effects (font (size 1.27 1.27)) (hide yes)))
+		(pin "1")
 	)
 	(wire (pts (xy 139.7 86.36) (xy 137.16 86.36))
@@
 		(property "Datasheet" "" (at 95.25 119.38 0)
 			(effects (font (size 1.27 1.27)) (hide yes)))
-		(property "Note" "ICHG=890/1.78k≈0.5A=0.17C@3000mAh，1%" (at 95.25 119.38 0)
-			(effects (font (size 1.27 1.27)) (hide yes)))
-		(pin "1")
-		(pin "2")
-	)
-	(symbol (lib_id "Device:R") (at 95.25 139.7 0) (unit 1)
-		(exclude_from_sim no) (in_bom yes) (on_board yes) (dnp no) (fields_autoplaced yes)
-		(property "Reference" "R10" (at 95.25 134.62 0)
-			(effects (font (size 1.27 1.27))))
-		(property "Value" "47k" (at 95.25 144.78 0)
-			(effects (font (size 1.27 1.27))))
-		(property "Footprint" "Resistor_SMD:R_0603_1608Metric" (at 95.25 139.7 0)
-			(effects (font (size 1.27 1.27)) (hide yes)))
-		(property "Datasheet" "" (at 95.25 139.7 0)
-			(effects (font (size 1.27 1.27)) (hide yes)))
-		(property "Note" "R_TMR：6.25h 安全定时，必须装（默认 5h 不够充满 3000mAh）" (at 95.25 139.7 0)
+		(property "Note" "ICHG=890/1.78k≈0.5A=0.05C@10000mAh，1%" (at 95.25 119.38 0)
 			(effects (font (size 1.27 1.27)) (hide yes)))
 		(pin "1")
@@
 		(property "LCSC" "C131337" (at 203.2 71.12 0)
 			(effects (font (size 1.27 1.27)) (hide yes)))
-		(property "Note" "pin1=电池+  pin2=GND（⚠️ 极性不可反）" (at 203.2 71.12 0)
+		(property "Note" "pin1=电池+  pin2=GND（极性不可反）；须接 1S2P 单 PCM 电池包 10000mAh" (at 203.2 71.12 0)
 			(effects (font (size 1.27 1.27)) (hide yes)))
 		(pin "1")
@@
 		(effects (font (size 1.27 1.27)) (justify left bottom))
 )
-	(text "【取值依据】U1=BQ24072RGT。ICHG = 890 / R_ISET = 0.5 A（=0.17C @3000mAh）；EN2=0 且 EN1=1 选 USB500 档（输入上限 500 mA）；~CE 接 VSS 常开；TD 接 VSS 使能充电终止；TS 经 10k 到 VSS 禁用温度监测；TMR 装 47k（6.25h 安全定时，默认 5h 不够）；VBUS 经 F1（500mA）后进 IN。取值与社区成熟方案对照见 docs/power-architecture.md 3.4" (exclude_from_sim no) (at 25.4 165.1 0)
+	(text "【取值依据】U1=BQ24072RGT。电池 = 2x5000mAh 并联（1S2P 共用一块 PCM，共 10000mAh）。ICHG = 890 / R_ISET = 0.5 A（=0.05C @10000mAh）；EN2=0 且 EN1=1 选 USB500 档（输入上限 500 mA）；~CE 接 VSS 常开；TD 接 VSS 使能充电终止；TS 经 10k 到 VSS 禁用温度监测；TMR 接 VSS 禁用所有安全定时器（充满 10000mAh 约需 20h，超出定时器 12h 上限）。VBUS 经 F1（500mA）后进 IN。容量与商用键盘对照见 docs/power-architecture.md 3.5" (exclude_from_sim no) (at 25.4 165.1 0)
 		(effects (font (size 1.27 1.27)) (justify left bottom))
 )
@@
 		(effects (font (size 1.27 1.27)) (justify left bottom))
 )
-	(text "【连接器约束】J2 为 JST-PH 2.0，额定 2 A（限 AWG #24 条件）。RGB 全亮峰值约 2.4 A 超过该额定，不可靠接插件承载全亮电流；pigtail 请指定 AWG #24" (exclude_from_sim no) (at 25.4 191.77 0)
+	(text "【电池与连接器约束】J2 为 JST-PH 2.0，额定 2 A（限 AWG #24 条件）。RGB 全亮峰值约 2.4 A 超过该额定，pigtail 请指定 AWG #24。电池须为 1S2P 一体化包（两块 5000mAh 共用一块 PCM），不可用两块各自带保护板的电芯直接并联（会互充，且两块保护板阈值失配）；PCM 的过流保护阈值必须大于 2A，否则 RGB 全亮会触发保护断电" (exclude_from_sim no) (at 25.4 191.77 0)
 		(effects (font (size 1.27 1.27)) (justify left bottom))
 )
@@
 		(effects (font (size 1.27 1.27)) (justify left bottom))
 )
-	(text "【投板后必须实测】1) AO3401A 在 Vgs 约 -0.9 V 时的关断漏电（标 UNVERIFIED）2) RGB 峰值电流下 OUT 压降是否仍在 250 mV 以内 3) 深睡整机电流（目标约 20 uA）" (exclude_from_sim no) (at 25.4 218.44 0)
-		(effects (font (size 1.27 1.27)) (justify left bottom))
-)
+	(text "【投板后必须实测】1) AO3401A 在 Vgs 约 -0.9 V 时的关断漏电（标 UNVERIFIED）2) RGB 峰值电流下 OUT 压降是否仍在 250 mV 以内 3) 深睡整机电流（目标约 20 uA）4) TMR 接 VSS 后充电能否正常走到 4.2 V 并靠终止电流判据结束（安全定时器已禁用）" (exclude_from_sim no) (at 25.4 218.44 0)
+		(effects (font (size 1.27 1.27)) (justify left bottom))
+)
