File: hardware/pcb/StarShield/power/power.kicad_sch (KiCad schematic)
At the start: 19 parts, among them J1 USB_C_Receptacle_USB2.0_16P, J2 B2B-PH-K-S, Q1 AO3401A, Q2 2N7002, U1 BQ24072RGT

Commit message: feat(power): P13 定案 —— 充电档位切到 ILIM 档 1.0A（含连带修正 F1 保险丝）
【决策】用户 2026-09-18 选定方案 2：EN2=OUT / EN1=GND（ILIM 档）、R_ILIM 1.6kΩ（输入限流 ≈1.0A）、R_ISET 887Ω（ICHG ≈1.0A = 0.10C）、充满约 10h。

【依据】商用同容量（≥5000mAh）键盘实测充电区间 0.035-0.163C（AULA L99 8000mAh/1300mA、Kzzi 10000mAh/1400mA、EPOMAKER TH87 10000mAh/<=1000mA、Hola87 10000mAh/350mA）；旧值 485mA = 0.049C 落在下三分之一。另有整机拆解实证：商用无线键盘用 TP4056（线性，最大 1A），且即使第 1 脚支持 TEMP 温测，厂商仍用 2 线电池包。

【连带修正 F1】原 500mA 保险丝是配 USB500 档的；输入切到 1.0A 后它会必然熔断 => 改为 1.5A（1.0A 工作电流约为额定的 67%）。这是改档位时发现的连带影响。

【BQ24072 约束核对】耗散 (5-3.7)x1.0 = 1.3W；按 JEDEC 板 RθJA=44.5°C/W 估 Tj ≈ 83°C，低于 125°C 热调节门限。定时器仍接 VSS 禁用（10h 仍压在 7.2-12h 的边缘，不赌芯片个体差异）。

【代价写明】这是本项目唯一主动超出 USB-C 声明之处（5.1kΩ 只声明 500mA，取 1.0A 超 2 倍）。商用产品普遍如此（AULA/Kzzi/EPOMAKER 都超），靠手册「勿用快充充电器」警告兜底。

【落地】power_design.py：U1.5->OUT、U1.6->GND、R3 1.6kΩ、R4 887Ω、F1 1.5A + 注释与 NOTES 全面更新；verify_power.py 具名断言同步（EN2=OUT/EN1=GND => ILIM 档；ISET 887Ω => 1.0A）。文档：power-architecture.md（3.1 四行 / 3 表 / 3.2 表格与理由 / 3.5.3 路线 / 5.2 / 6 P13 关闭）、decisions.md、controller-and-battery-facts.md 2.3、bq24072-pinout.md 3.5、ADR-0002 勘误、handoff 9/12。

【验收】19 元件 / 70 条引脚连接；四校验器全绿；两轮生成器哈希一致；ERC 仍 0 error / 2 warning。
Parts:
- F1: value 500mA -> 1.5A; Note USB 输入限流保险丝；额定值待按降额曲线复核 -> USB 输入保险丝：1.0A 工作电流下选 1.5A；待按降额曲线复核
- R3: value 1.5k -> 1.6k; Note USB500 档下不参与限流，但必须装（悬空=关闭充电）；取值同社区 1.5k -> ILIM 档：输入限流 1610/1.6k≈1.0A；悬空=关闭充电，必须装
- R4: value 1.78k -> 887; Note ICHG=890/1.78k≈0.5A=0.05C@10000mAh，1% -> ICHG=890/887≈1.0A=0.10C@10000mAh，1%
Connections:
- net GND: now also U1.6 (EN1); no longer U1.5 (EN2)
- net OUT: now also U1.5 (EN2); no longer U1.6 (EN1)
Other:
- note added: "【取值依据】U1=BQ24072RGT。电池 = 2x5000mAh 并联（1S2P 共用一块 PCM，共 10000mAh）。ICHG = 890 / R_ISET = 1.0 A（=0.10C @10000mAh）；EN2=1 且 EN1=0 选 ILIM 档，输入限流 = 1610 / R_ILIM = 1.0 A；~CE 接 VSS 常开；TD 接 VSS 使能充电终止；TS 经 10k 到 VSS 禁用温度监测；TMR 接 VSS 禁用所有安全定时器（10h 仍超定时器 typ 9.6h）。VBUS 经 F1（1.5A）后进 IN。注意：输入取 1.0A 超出 5.1k 的 USB 声明，是有意取舍，见 docs/power-architecture.md 3.7"
- note added: "【本版留空 / 未决项】USB-C 的 D+ D- SBU1 SBU2 全部 NC（J1 只做充电 —— nRF52840 的 USB 是独立专用引脚，nice!nano 排针上无引出）；U1 的 ~PGOOD 悬空（预留测试点）。F1 保险丝额定值待按所选料号降额曲线复核（P15）。详见 docs/power-architecture.md 第 6 节待办"
- note removed: "【取值依据】U1=BQ24072RGT。电池 = 2x5000mAh 并联（1S2P 共用一块 PCM，共 10000mAh）。ICHG = 890 / R_ISET = 0.5 A（=0.05C @10000mAh）；EN2=0 且 EN1=1 选 USB500 档（输入上限 500 mA）；~CE 接 VSS 常开；TD 接 VSS 使能充电终止；TS 经 10k 到 VSS 禁用温度监测；TMR 接 VSS 禁用所有安全定时器（充满 10000mAh 约需 20.6h，超出定时器 7.2-12h 上限）。VBUS 经 F1（500mA）后进 IN。容量与商用键盘对照见 docs/power-architecture.md 3.5"
- note removed: "【本版留空 / 未决项】P2 与 P10：USB-C 的 D+ D- SBU 全部 NC（第一版 USB-C 仅充电）；U1 的 ~PGOOD 悬空（预留测试点）。F1 保险丝的额定值待按所选料号的降额曲线复核。详见 docs/power-architecture.md 第 6 节待办"
Changed lines of the file:
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@@
 	(wire (pts (xy 139.7 99.06) (xy 137.16 99.06))
 		(stroke (width 0) (type default)))
-	(symbol (lib_id "power:GND") (at 137.16 99.06 270) (unit 1)
-		(exclude_from_sim no) (in_bom yes) (on_board yes) (dnp no) (fields_autoplaced yes)
-		(property "Reference" "#PWR0188" (at 137.16 93.98 0)
-			(effects (font (size 1.27 1.27)) (hide yes)))
-		(property "Value" "GND" (at 137.16 104.14 0)
-			(effects (font (size 1.27 1.27)) (hide yes)))
-		(property "Footprint" "" (at 137.16 99.06 0)
-			(effects (font (size 1.27 1.27)) (hide yes)))
-		(property "Datasheet" "" (at 137.16 99.06 0)
-			(effects (font (size 1.27 1.27)) (hide yes)))
-		(pin "1")
+	(global_label "OUT" (shape passive) (at 137.16 99.06 180) (fields_autoplaced yes)
+		(effects (font (size 1.27 1.27)) (justify right))
 	)
 	(wire (pts (xy 139.7 96.52) (xy 137.16 96.52))
 		(stroke (width 0) (type default)))
-	(global_label "OUT" (shape passive) (at 137.16 96.52 180) (fields_autoplaced yes)
-		(effects (font (size 1.27 1.27)) (justify right))
+	(symbol (lib_id "power:GND") (at 137.16 96.52 270) (unit 1)
+		(exclude_from_sim no) (in_bom yes) (on_board yes) (dnp no) (fields_autoplaced yes)
+		(property "Reference" "#PWR0188" (at 137.16 91.44 0)
+			(effects (font (size 1.27 1.27)) (hide yes)))
+		(property "Value" "GND" (at 137.16 101.6 0)
+			(effects (font (size 1.27 1.27)) (hide yes)))
+		(property "Footprint" "" (at 137.16 96.52 0)
+			(effects (font (size 1.27 1.27)) (hide yes)))
+		(property "Datasheet" "" (at 137.16 96.52 0)
+			(effects (font (size 1.27 1.27)) (hide yes)))
+		(pin "1")
 	)
 	(no_connect (at 165.1 104.14))
@@
 		(property "Reference" "F1" (at 134.62 66.04 0)
 			(effects (font (size 1.27 1.27))))
-		(property "Value" "500mA" (at 134.62 76.2 0)
+		(property "Value" "1.5A" (at 134.62 76.2 0)
 			(effects (font (size 1.27 1.27))))
 		(property "Footprint" "Fuse:Fuse_0603_1608Metric" (at 134.62 71.12 0)
@@
 		(property "Datasheet" "" (at 134.62 71.12 0)
 			(effects (font (size 1.27 1.27)) (hide yes)))
-		(property "Note" "USB 输入限流保险丝；额定值待按降额曲线复核" (at 134.62 71.12 0)
+		(property "Note" "USB 输入保险丝：1.0A 工作电流下选 1.5A；待按降额曲线复核" (at 134.62 71.12 0)
 			(effects (font (size 1.27 1.27)) (hide yes)))
 		(pin "1")
@@
 		(property "Reference" "R3" (at 95.25 93.98 0)
 			(effects (font (size 1.27 1.27))))
-		(property "Value" "1.5k" (at 95.25 104.14 0)
+		(property "Value" "1.6k" (at 95.25 104.14 0)
 			(effects (font (size 1.27 1.27))))
 		(property "Footprint" "Resistor_SMD:R_0603_1608Metric" (at 95.25 99.06 0)
@@
 		(property "Datasheet" "" (at 95.25 99.06 0)
 			(effects (font (size 1.27 1.27)) (hide yes)))
-		(property "Note" "USB500 档下不参与限流，但必须装（悬空=关闭充电）；取值同社区 1.5k" (at 95.25 99.06 0)
+		(property "Note" "ILIM 档：输入限流 1610/1.6k≈1.0A；悬空=关闭充电，必须装" (at 95.25 99.06 0)
 			(effects (font (size 1.27 1.27)) (hide yes)))
 		(pin "1")
@@
 		(property "Reference" "R4" (at 95.25 114.3 0)
 			(effects (font (size 1.27 1.27))))
-		(property "Value" "1.78k" (at 95.25 124.46 0)
+		(property "Value" "887" (at 95.25 124.46 0)
 			(effects (font (size 1.27 1.27))))
 		(property "Footprint" "Resistor_SMD:R_0603_1608Metric" (at 95.25 119.38 0)
@@
 		(property "Datasheet" "" (at 95.25 119.38 0)
 			(effects (font (size 1.27 1.27)) (hide yes)))
-		(property "Note" "ICHG=890/1.78k≈0.5A=0.05C@10000mAh，1%" (at 95.25 119.38 0)
+		(property "Note" "ICHG=890/887≈1.0A=0.10C@10000mAh，1%" (at 95.25 119.38 0)
 			(effects (font (size 1.27 1.27)) (hide yes)))
 		(pin "1")
@@
 		(effects (font (size 1.27 1.27)) (justify left bottom))
 )
-	(text "【取值依据】U1=BQ24072RGT。电池 = 2x5000mAh 并联（1S2P 共用一块 PCM，共 10000mAh）。ICHG = 890 / R_ISET = 0.5 A（=0.05C @10000mAh）；EN2=0 且 EN1=1 选 USB500 档（输入上限 500 mA）；~CE 接 VSS 常开；TD 接 VSS 使能充电终止；TS 经 10k 到 VSS 禁用温度监测；TMR 接 VSS 禁用所有安全定时器（充满 10000mAh 约需 20.6h，超出定时器 7.2-12h 上限）。VBUS 经 F1（500mA）后进 IN。容量与商用键盘对照见 docs/power-architecture.md 3.5" (exclude_from_sim no) (at 25.4 165.1 0)
+	(text "【取值依据】U1=BQ24072RGT。电池 = 2x5000mAh 并联（1S2P 共用一块 PCM，共 10000mAh）。ICHG = 890 / R_ISET = 1.0 A（=0.10C @10000mAh）；EN2=1 且 EN1=0 选 ILIM 档，输入限流 = 1610 / R_ILIM = 1.0 A；~CE 接 VSS 常开；TD 接 VSS 使能充电终止；TS 经 10k 到 VSS 禁用温度监测；TMR 接 VSS 禁用所有安全定时器（10h 仍超定时器 typ 9.6h）。VBUS 经 F1（1.5A）后进 IN。注意：输入取 1.0A 超出 5.1k 的 USB 声明，是有意取舍，见 docs/power-architecture.md 3.7" (exclude_from_sim no) (at 25.4 165.1 0)
 		(effects (font (size 1.27 1.27)) (justify left bottom))
 )
@@
 		(effects (font (size 1.27 1.27)) (justify left bottom))
 )
-	(text "【本版留空 / 未决项】P2 与 P10：USB-C 的 D+ D- SBU 全部 NC（第一版 USB-C 仅充电）；U1 的 ~PGOOD 悬空（预留测试点）。F1 保险丝的额定值待按所选料号的降额曲线复核。详见 docs/power-architecture.md 第 6 节待办" (exclude_from_sim no) (at 25.4 209.55 0)
+	(text "【本版留空 / 未决项】USB-C 的 D+ D- SBU1 SBU2 全部 NC（J1 只做充电 —— nRF52840 的 USB 是独立专用引脚，nice!nano 排针上无引出）；U1 的 ~PGOOD 悬空（预留测试点）。F1 保险丝额定值待按所选料号降额曲线复核（P15）。详见 docs/power-architecture.md 第 6 节待办" (exclude_from_sim no) (at 25.4 209.55 0)
 		(effects (font (size 1.27 1.27)) (justify left bottom))
 )

Commit message: feat(power): P15 定案 —— F1 改为 2A hold 自恢复保险丝（1812 封装，MF-MSMF200）
1.5A 档被降额曲线否决：MF-MSMF150 在 60°C 时 Ihold 仅 1.00A，等于工作电流（零余量），
70°C 时 0.88A 会误断。2A 档 60°C 仍 1.50A（余量 50%）。压降最大 80mV 不影响充电。
类型改 PTC（新手免换件），封装 0603 → 1812。LCSC 料号留待 BOM。
Parts:
- F1: value 1.5A -> 2A; footprint Fuse:Fuse_0603_1608Metric -> Fuse:Fuse_1812_4532Metric; LCSC (none) -> ❓待补（BOM 阶段）; MPN (none) -> MF-MSMF200; Note USB 输入保险丝：1.0A 工作电流下选 1.5A；待按降额曲线复核 -> USB 输入自恢复保险丝：hold 2.0A/trip 4.0A/8V/1812；60°C 降额后仍 1.50A
Other:
- note added: "【取值依据】U1=BQ24072RGT。电池 = 2x5000mAh 并联（1S2P 共用一块 PCM，共 10000mAh）。ICHG = 890 / R_ISET = 1.0 A（=0.10C @10000mAh）；EN2=1 且 EN1=0 选 ILIM 档，输入限流 = 1610 / R_ILIM = 1.0 A；~CE 接 VSS 常开；TD 接 VSS 使能充电终止；TS 经 10k 到 VSS 禁用温度监测；TMR 接 VSS 禁用所有安全定时器（10h 仍超定时器 typ 9.6h）。VBUS 经 F1（2A hold 自恢复保险丝，1812）后进 IN。注意：输入取 1.0A 超出 5.1k 的 USB 声明，是有意取舍，见 docs/power-architecture.md 3.7"
- note added: "【本版留空 / 未决项】USB-C 的 D+ D- SBU1 SBU2 全部 NC（J1 只做充电 —— nRF52840 的 USB 是独立专用引脚，nice!nano 排针上无引出）；U1 的 ~PGOOD 悬空（预留测试点）。F1 已按降额曲线定案为 2A hold 的 1812 自恢复保险丝（1.5A 档在 60°C 降额后仅 1.00A，等于工作电流，会误断）。详见 docs/power-architecture.md 第 6 节待办"
- note removed: "【取值依据】U1=BQ24072RGT。电池 = 2x5000mAh 并联（1S2P 共用一块 PCM，共 10000mAh）。ICHG = 890 / R_ISET = 1.0 A（=0.10C @10000mAh）；EN2=1 且 EN1=0 选 ILIM 档，输入限流 = 1610 / R_ILIM = 1.0 A；~CE 接 VSS 常开；TD 接 VSS 使能充电终止；TS 经 10k 到 VSS 禁用温度监测；TMR 接 VSS 禁用所有安全定时器（10h 仍超定时器 typ 9.6h）。VBUS 经 F1（1.5A）后进 IN。注意：输入取 1.0A 超出 5.1k 的 USB 声明，是有意取舍，见 docs/power-architecture.md 3.7"
- note removed: "【本版留空 / 未决项】USB-C 的 D+ D- SBU1 SBU2 全部 NC（J1 只做充电 —— nRF52840 的 USB 是独立专用引脚，nice!nano 排针上无引出）；U1 的 ~PGOOD 悬空（预留测试点）。F1 保险丝额定值待按所选料号降额曲线复核（P15）。详见 docs/power-architecture.md 第 6 节待办"
Changed lines of the file:
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@@
 		(property "Reference" "F1" (at 134.62 66.04 0)
 			(effects (font (size 1.27 1.27))))
-		(property "Value" "1.5A" (at 134.62 76.2 0)
-			(effects (font (size 1.27 1.27))))
-		(property "Footprint" "Fuse:Fuse_0603_1608Metric" (at 134.62 71.12 0)
+		(property "Value" "2A" (at 134.62 76.2 0)
+			(effects (font (size 1.27 1.27))))
+		(property "Footprint" "Fuse:Fuse_1812_4532Metric" (at 134.62 71.12 0)
 			(effects (font (size 1.27 1.27)) (hide yes)))
 		(property "Datasheet" "" (at 134.62 71.12 0)
 			(effects (font (size 1.27 1.27)) (hide yes)))
-		(property "Note" "USB 输入保险丝：1.0A 工作电流下选 1.5A；待按降额曲线复核" (at 134.62 71.12 0)
+		(property "MPN" "MF-MSMF200" (at 134.62 71.12 0)
+			(effects (font (size 1.27 1.27)) (hide yes)))
+		(property "LCSC" "❓待补（BOM 阶段）" (at 134.62 71.12 0)
+			(effects (font (size 1.27 1.27)) (hide yes)))
+		(property "Note" "USB 输入自恢复保险丝：hold 2.0A/trip 4.0A/8V/1812；60°C 降额后仍 1.50A" (at 134.62 71.12 0)
 			(effects (font (size 1.27 1.27)) (hide yes)))
 		(pin "1")
@@
 		(effects (font (size 1.27 1.27)) (justify left bottom))
 )
-	(text "【取值依据】U1=BQ24072RGT。电池 = 2x5000mAh 并联（1S2P 共用一块 PCM，共 10000mAh）。ICHG = 890 / R_ISET = 1.0 A（=0.10C @10000mAh）；EN2=1 且 EN1=0 选 ILIM 档，输入限流 = 1610 / R_ILIM = 1.0 A；~CE 接 VSS 常开；TD 接 VSS 使能充电终止；TS 经 10k 到 VSS 禁用温度监测；TMR 接 VSS 禁用所有安全定时器（10h 仍超定时器 typ 9.6h）。VBUS 经 F1（1.5A）后进 IN。注意：输入取 1.0A 超出 5.1k 的 USB 声明，是有意取舍，见 docs/power-architecture.md 3.7" (exclude_from_sim no) (at 25.4 165.1 0)
+	(text "【取值依据】U1=BQ24072RGT。电池 = 2x5000mAh 并联（1S2P 共用一块 PCM，共 10000mAh）。ICHG = 890 / R_ISET = 1.0 A（=0.10C @10000mAh）；EN2=1 且 EN1=0 选 ILIM 档，输入限流 = 1610 / R_ILIM = 1.0 A；~CE 接 VSS 常开；TD 接 VSS 使能充电终止；TS 经 10k 到 VSS 禁用温度监测；TMR 接 VSS 禁用所有安全定时器（10h 仍超定时器 typ 9.6h）。VBUS 经 F1（2A hold 自恢复保险丝，1812）后进 IN。注意：输入取 1.0A 超出 5.1k 的 USB 声明，是有意取舍，见 docs/power-architecture.md 3.7" (exclude_from_sim no) (at 25.4 165.1 0)
 		(effects (font (size 1.27 1.27)) (justify left bottom))
 )
@@
 		(effects (font (size 1.27 1.27)) (justify left bottom))
 )
-	(text "【本版留空 / 未决项】USB-C 的 D+ D- SBU1 SBU2 全部 NC（J1 只做充电 —— nRF52840 的 USB 是独立专用引脚，nice!nano 排针上无引出）；U1 的 ~PGOOD 悬空（预留测试点）。F1 保险丝额定值待按所选料号降额曲线复核（P15）。详见 docs/power-architecture.md 第 6 节待办" (exclude_from_sim no) (at 25.4 209.55 0)
-		(effects (font (size 1.27 1.27)) (justify left bottom))
-)
+	(text "【本版留空 / 未决项】USB-C 的 D+ D- SBU1 SBU2 全部 NC（J1 只做充电 —— nRF52840 的 USB 是独立专用引脚，nice!nano 排针上无引出）；U1 的 ~PGOOD 悬空（预留测试点）。F1 已按降额曲线定案为 2A hold 的 1812 自恢复保险丝（1.5A 档在 60°C 降额后仅 1.00A，等于工作电流，会误断）。详见 docs/power-architecture.md 第 6 节待办" (exclude_from_sim no) (at 25.4 209.55 0)
+		(effects (font (size 1.27 1.27)) (justify left bottom))
+)

Commit message: fix(schematic): 三处地基修复 —— 矩阵跨图标签、充电 LED 位号冲突、网表校验盲区
1. 矩阵 ROW/COL 由局部标签改为全局标签：KiCad 局部标签不跨 sheet 相连，
   三张矩阵子图的同名 COL 在真实网表里带各自路径前缀、互不相连；
   该缺陷曾被「单图导出+按名合并」的旧校验掩盖。
2. verify_netlist.py 改为从根图整体导出网表校验（校验真实连通性）；
   列网节点数断言同步为 95 键 + 18 个 595 驱动端 = 113。
3. 充电 LED 位号 D1 -> D96：与矩阵二极管 D1 冲突（根图整体网表
   元件数 208 != 209 暴露）；D96 = 矩阵 D1..D95 顺延，避开将来 RGB 子图 LED1..95。
verify_power / verify_netlist 全绿。
Parts:
- removed D1: RED, LED_SMD:LED_0603_1608Metric, symbol Device:LED
- added D96: RED, LED_SMD:LED_0603_1608Metric, symbol Device:LED
Connections:
- net CHG_LED_A: now also D96.2 (A)
- net nCHG: now also D96.1 (K)
Changed lines of the file:
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@@
 	(symbol (lib_id "Device:LED") (at 185.42 121.92 0) (unit 1)
 		(exclude_from_sim no) (in_bom yes) (on_board yes) (dnp no) (fields_autoplaced yes)
-		(property "Reference" "D1" (at 185.42 116.84 0)
+		(property "Reference" "D96" (at 185.42 116.84 0)
 			(effects (font (size 1.27 1.27))))
 		(property "Value" "RED" (at 185.42 127.0 0)

Commit message: feat(power): 方案①落地 —— 模块 B+/RAW 由 OUT 改接 VBAT（插模块口即充电）；模块整组左移 + J1 让位
背景（用户质疑成立）：商业键盘一律「一个口 = 数据 + 充电」（Kisnt KN85 / 雷柏 V700-8A /
CHERRY KW 9200 官方口径）；社区 nice!nano 方案把电池挂在模块自带充电器输出上，插模块口即充电。
我们原先把电池接自研 BQ24072 的 BAT、模块挂 OUT ⇒ 模块充电器的电流进不了电池
（OUT→BAT 不是充电路径）⇒ 有线模式下充不上电。

改动：
- 电路：J3B 孔1/孔2（B+/RAW）网络 OUT -> VBAT；VBAT 由电源子图局部网升为跨子图全局网
  （power_design.py 与 control_design.py 的 GLOBAL_NETS 各加 VBAT）
- 子图：power.kicad_sch / control.kicad_sch 重生成（版式自检通过）
- 校验：verify_control 断言改为「VBAT 跨图连通（J3B 孔1/2 + U1/J2/C3）」+
  「OUT 不再挂 J3B」；网表类五项校验全绿
- 几何（B6-2）：nice!nano 插座整组左移 30.46 mm（孔1 x=7.00、口面 x=1.70 与壳面齐平）；
  J1/R1/R2/F1 让位到 x=155-168；pcb_design.py 同步
- 板文件：J3B 孔1/2 改网为 VBAT（旧 OUT 走线已随左移一并清除）
- 文档：power-architecture.md §1 / bq24072-pinout.md §2.3 / decisions.md 电源段各加「重载仍接 OUT、
  模块为唯一例外」的修订说明；量测文档 §6.6 记录完整对标与代价

⚠️ 遗留（下一步）：肩部走线缺口待补（左移时删了 76 项），Freerouting 正在用新网表全板重布；
完成后需重跑 DRC + 七项校验器。
Other:
- note added: "【电源路径】重载（VLED 灯轨等）必须接 OUT 而不是 BAT（ADR-0002）。OUT 稳压到 VBAT + 225 mV，满电时 OUT 约 4.4 V。VLED 由 OUT 经 Q1 门控 —— 属电池直供，不含任何升压（ADR-0007 / ADR-0005）。⚠️ 2026-09-19 例外：nice!nano 模块的 B+/RAW 改接 VBAT（不再接 OUT）—— 因为模块自带充电器要能把电流送进电池（插模块口即充电）；模块本身电流很小（休眠 20uA 级），不影响电源路径的意义"
- note removed: "【电源路径】负载必须接 OUT 而不是 BAT（ADR-0002）。OUT 稳压到 VBAT + 225 mV，满电时 OUT 约 4.4 V。VLED 由 OUT 经 Q1 门控 —— 属电池直供，不含任何升压（ADR-0007 / ADR-0005）"
Changed lines of the file:
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@@
 	(wire (pts (xy 185.42 74.93) (xy 185.42 72.39))
 		(stroke (width 0) (type default)))
-	(label "VBAT" (at 185.42 72.39 90) (fields_autoplaced yes)
-		(effects (font (size 1.27 1.27)) (justify left bottom))
+	(global_label "VBAT" (shape passive) (at 185.42 72.39 90) (fields_autoplaced yes)
+		(effects (font (size 1.27 1.27)) (justify left))
 	)
 	(wire (pts (xy 185.42 82.55) (xy 185.42 85.09))
@@
 	(wire (pts (xy 165.1 93.98) (xy 167.64 93.98))
 		(stroke (width 0) (type default)))
-	(label "VBAT" (at 167.64 93.98 0) (fields_autoplaced yes)
-		(effects (font (size 1.27 1.27)) (justify left bottom))
+	(global_label "VBAT" (shape passive) (at 167.64 93.98 0) (fields_autoplaced yes)
+		(effects (font (size 1.27 1.27)) (justify left))
 	)
 	(wire (pts (xy 139.7 91.44) (xy 137.16 91.44))
@@
 	(wire (pts (xy 198.12 71.12) (xy 195.58 71.12))
 		(stroke (width 0) (type default)))
-	(label "VBAT" (at 195.58 71.12 180) (fields_autoplaced yes)
-		(effects (font (size 1.27 1.27)) (justify right bottom))
+	(global_label "VBAT" (shape passive) (at 195.58 71.12 180) (fields_autoplaced yes)
+		(effects (font (size 1.27 1.27)) (justify right))
 	)
 	(wire (pts (xy 198.12 73.66) (xy 195.58 73.66))
@@
 		(effects (font (size 1.27 1.27)) (justify left bottom))
 )
-	(text "【电源路径】负载必须接 OUT 而不是 BAT（ADR-0002）。OUT 稳压到 VBAT + 225 mV，满电时 OUT 约 4.4 V。VLED 由 OUT 经 Q1 门控 —— 属电池直供，不含任何升压（ADR-0007 / ADR-0005）" (exclude_from_sim no) (at 25.4 173.99 0)
+	(text "【电源路径】重载（VLED 灯轨等）必须接 OUT 而不是 BAT（ADR-0002）。OUT 稳压到 VBAT + 225 mV，满电时 OUT 约 4.4 V。VLED 由 OUT 经 Q1 门控 —— 属电池直供，不含任何升压（ADR-0007 / ADR-0005）。⚠️ 2026-09-19 例外：nice!nano 模块的 B+/RAW 改接 VBAT（不再接 OUT）—— 因为模块自带充电器要能把电流送进电池（插模块口即充电）；模块本身电流很小（休眠 20uA 级），不影响电源路径的意义" (exclude_from_sim no) (at 25.4 173.99 0)
 		(effects (font (size 1.27 1.27)) (justify left bottom))
 )
