File: hardware/pcb/StarShield/matrix/matrix_r012.kicad_sch (KiCad schematic)
At the start: 68 parts, among them SW1 Esc, SW10 F7, SW11 F8, SW12 F9, SW13 F10, SW14 F11, SW15 F12, SW16 Delete, SW17 /, SW18 *, SW19 -, SW2 FN, SW20 +, SW21 ~/`, SW22 !/1, SW23 @/2, SW24 #/3, SW25 $/4, SW26 %/5, SW27 ^/6, SW28 &/7, SW29 */8, SW3 Num Lock, SW30 (/9, SW31 )/0, SW32 _/-, SW33 +/=, SW34 Back Space, SW4 F1, SW5 F2, SW6 F3, SW7 F4, SW8 F5, SW9 F6

Commit message: feat(b3): 自画 MX 热插拔座封装（8 档），313/313 元件封装全部就位
B3 定案：自画（官方库没有热插拔座；社区库 daprice/keyswitches.pretty 的
Kailh_socket_MX 是 CC BY-SA 4.0、无官方库的「用于设计不受约束」例外，不可引入）。

- 新增 gen_footprints.py -> hardware/pcb/StarShield/footprints/StarShield.pretty/
  8 档：1.00 / 1.25 / 1.50 / 1.75 / 2.00 / 2.00u_Vertical / 2.25 / 6.25u。
- 做法：以官方 SW_Cherry_MX_<宽度>u_PCB 为基底（含轴体机械孔与**卫星轴 stabilizer
  孔位** —— 官方库没有独立 stabilizer 封装，这正是它按宽度分档的原因），
  只追加 2 个 B.Cu SMD 焊盘（Kailh socket 叶片），编号与官方 PTH 焊盘同为 1/2
  => 同 net、装配二选一（直焊 PTH / 热插拔 SMD；socket 焊背面、轴体正面插入）。
  一个坐标都不手抄：孔位与 stabilizer 间距全部来自官方文件。
- 矩阵 95 个开关按键宽选档（含阶梯 Enter 按 stabilizer 合并宽 2.25u、
  两个 1u x 2u 竖键用 2.00u_Vertical），与 matrix.json 键宽分布逐项吻合。
- verify_footprints.py 改为「先查工程自带库、再退回官方库」。
- 实测：313 / 313 个元件封装全部就位，0 缺失；五个校验器 + 根图 ERC 0 error。
⚠️ UNVERIFIED：socket 焊盘位置/孔径源自公开尺寸（非 Kailh 原厂手册），
   并入 B6 投板前实物核对；保留 PTH 焊盘是该风险的兜底。
Parts:
- SW1, SW10, SW11, SW12, SW13, SW14, SW15, SW16, SW17, SW18, SW19, SW2, SW20, SW21, SW22, SW23, SW24, SW25, SW26, SW27, SW28, SW29, SW3, SW30, SW31, SW32, SW33, SW4, SW5, SW6, SW7, SW8, SW9: footprint Button_Switch_Keyboard:SW_MX_Hotswap -> StarShield:SW_MX_Hotswap_Optional_1.00u
- SW34: footprint Button_Switch_Keyboard:SW_MX_Hotswap -> StarShield:SW_MX_Hotswap_Optional_2.00u
