File: hardware/pcb/StarShield/matrix/matrix_r234.kicad_sch (KiCad schematic)
At the start: 66 parts, among them SW35 Delete, SW36 7/Home, SW37 8/↑, SW38 9/PgUp, SW39 Tab, SW40 Q, SW41 W, SW42 E, SW43 R, SW44 T, SW45 Y, SW46 U, SW47 I, SW48 O, SW49 P, SW50 {/[, SW51 }/], SW52 Enter, SW53 4/←, SW54 5, SW55 6/→, SW56 Caps Lock, SW57 A, SW58 S, SW59 D, SW60 F, SW61 G, SW62 H, SW63 J, SW64 K, SW65 L, SW66 :/;, SW67 "/'

Commit message: feat(b3): 自画 MX 热插拔座封装（8 档），313/313 元件封装全部就位
B3 定案：自画（官方库没有热插拔座；社区库 daprice/keyswitches.pretty 的
Kailh_socket_MX 是 CC BY-SA 4.0、无官方库的「用于设计不受约束」例外，不可引入）。

- 新增 gen_footprints.py -> hardware/pcb/StarShield/footprints/StarShield.pretty/
  8 档：1.00 / 1.25 / 1.50 / 1.75 / 2.00 / 2.00u_Vertical / 2.25 / 6.25u。
- 做法：以官方 SW_Cherry_MX_<宽度>u_PCB 为基底（含轴体机械孔与**卫星轴 stabilizer
  孔位** —— 官方库没有独立 stabilizer 封装，这正是它按宽度分档的原因），
  只追加 2 个 B.Cu SMD 焊盘（Kailh socket 叶片），编号与官方 PTH 焊盘同为 1/2
  => 同 net、装配二选一（直焊 PTH / 热插拔 SMD；socket 焊背面、轴体正面插入）。
  一个坐标都不手抄：孔位与 stabilizer 间距全部来自官方文件。
- 矩阵 95 个开关按键宽选档（含阶梯 Enter 按 stabilizer 合并宽 2.25u、
  两个 1u x 2u 竖键用 2.00u_Vertical），与 matrix.json 键宽分布逐项吻合。
- verify_footprints.py 改为「先查工程自带库、再退回官方库」。
- 实测：313 / 313 个元件封装全部就位，0 缺失；五个校验器 + 根图 ERC 0 error。
⚠️ UNVERIFIED：socket 焊盘位置/孔径源自公开尺寸（非 Kailh 原厂手册），
   并入 B6 投板前实物核对；保留 PTH 焊盘是该风险的兜底。
Parts:
- SW35: footprint Button_Switch_Keyboard:SW_MX_Hotswap -> StarShield:SW_MX_Hotswap_Optional_2.00u_Vertical
- SW36, SW37, SW38, SW40, SW41, SW42, SW43, SW44, SW45, SW46, SW47, SW48, SW49, SW50, SW51, SW53, SW54, SW55, SW57, SW58, SW59, SW60, SW61, SW62, SW63, SW64, SW65, SW66, SW67: footprint Button_Switch_Keyboard:SW_MX_Hotswap -> StarShield:SW_MX_Hotswap_Optional_1.00u
- SW39: footprint Button_Switch_Keyboard:SW_MX_Hotswap -> StarShield:SW_MX_Hotswap_Optional_1.50u
- SW52: footprint Button_Switch_Keyboard:SW_MX_Hotswap -> StarShield:SW_MX_Hotswap_Optional_2.25u
- SW56: footprint Button_Switch_Keyboard:SW_MX_Hotswap -> StarShield:SW_MX_Hotswap_Optional_1.75u
