File: hardware/pcb/StarShield/matrix/matrix_r45.kicad_sch (KiCad schematic)
At the start: 56 parts, among them SW68 Enter, SW69 1/End, SW70 2/↓, SW71 3/PgDn, SW72 Shift, SW73 Z, SW74 X, SW75 C, SW76 V, SW77 B, SW78 N, SW79 M, SW80 </,, SW81 >/., SW82 ?//, SW83 ↑, SW84 Shift, SW85 0/Ins, SW86 ./Del, SW87 Ctrl, SW88 Win, SW89 Alt, SW90 Space, SW91 |/\, SW92 ←, SW93 ↓, SW94 →, SW95 Ctrl

Commit message: feat(b3): 自画 MX 热插拔座封装（8 档），313/313 元件封装全部就位
B3 定案：自画（官方库没有热插拔座；社区库 daprice/keyswitches.pretty 的
Kailh_socket_MX 是 CC BY-SA 4.0、无官方库的「用于设计不受约束」例外，不可引入）。

- 新增 gen_footprints.py -> hardware/pcb/StarShield/footprints/StarShield.pretty/
  8 档：1.00 / 1.25 / 1.50 / 1.75 / 2.00 / 2.00u_Vertical / 2.25 / 6.25u。
- 做法：以官方 SW_Cherry_MX_<宽度>u_PCB 为基底（含轴体机械孔与**卫星轴 stabilizer
  孔位** —— 官方库没有独立 stabilizer 封装，这正是它按宽度分档的原因），
  只追加 2 个 B.Cu SMD 焊盘（Kailh socket 叶片），编号与官方 PTH 焊盘同为 1/2
  => 同 net、装配二选一（直焊 PTH / 热插拔 SMD；socket 焊背面、轴体正面插入）。
  一个坐标都不手抄：孔位与 stabilizer 间距全部来自官方文件。
- 矩阵 95 个开关按键宽选档（含阶梯 Enter 按 stabilizer 合并宽 2.25u、
  两个 1u x 2u 竖键用 2.00u_Vertical），与 matrix.json 键宽分布逐项吻合。
- verify_footprints.py 改为「先查工程自带库、再退回官方库」。
- 实测：313 / 313 个元件封装全部就位，0 缺失；五个校验器 + 根图 ERC 0 error。
⚠️ UNVERIFIED：socket 焊盘位置/孔径源自公开尺寸（非 Kailh 原厂手册），
   并入 B6 投板前实物核对；保留 PTH 焊盘是该风险的兜底。
Parts:
- SW68: footprint Button_Switch_Keyboard:SW_MX_Hotswap -> StarShield:SW_MX_Hotswap_Optional_2.00u_Vertical
- SW69, SW70, SW71, SW73, SW74, SW75, SW76, SW77, SW78, SW79, SW80, SW81, SW82, SW83, SW91, SW92, SW93, SW94, SW95: footprint Button_Switch_Keyboard:SW_MX_Hotswap -> StarShield:SW_MX_Hotswap_Optional_1.00u
- SW72: footprint Button_Switch_Keyboard:SW_MX_Hotswap -> StarShield:SW_MX_Hotswap_Optional_2.25u
- SW84: footprint Button_Switch_Keyboard:SW_MX_Hotswap -> StarShield:SW_MX_Hotswap_Optional_1.75u
- SW85, SW86: footprint Button_Switch_Keyboard:SW_MX_Hotswap -> StarShield:SW_MX_Hotswap_Optional_1.50u
- SW87, SW88, SW89: footprint Button_Switch_Keyboard:SW_MX_Hotswap -> StarShield:SW_MX_Hotswap_Optional_1.25u
- SW90: footprint Button_Switch_Keyboard:SW_MX_Hotswap -> StarShield:SW_MX_Hotswap_Optional_6.25u
