File: hardware/pcb/StarShield/Starshield-plate.kicad_pcb (KiCad board)
At the start: 2 copper layers, 374.7 x 127.1 mm, 103 parts

Commit message: feat(pcb): USB-C 移左上角 / 三档开关移右上角；改为 4 层板
用户 2026-09-19 定的两处摆位：
- J1 (USB-C) 210,5.5 -> 15,5.5（左上角）；**R1/R2（CC 下拉）与 F1 随连接器左移**
  —— CC 走线必须短，否则是 USB-C 坏实践。代价：VBUS 从 F1 到 U1 变成约 230mm 长线
  （0.8mm 宽、1A，电气无碍）。
- SW96（三档模式开关）75,12 -> 360,6（右上角）。代价：MODE0/1/2 三条线从约 35mm
  变成约 320mm（μA 级信号，无碍）。

层数：2 -> **4 层**。⚠️ 关键教训：**层数属设计数据，必须由生成器产出** ——
先前用 MCP add_layer 加的 In1/In2 被下一次 gen_pcb.py 覆盖掉了。现写死进 gen_pcb.py 的
LAYERS，层号与顺序**照抄 KiCad 自己写出的形式**（B.Cu 的 id 是 2 而不是 31；
KiCad 还会去掉 F.SilkS/B.SilkS 的别名串）。

叠层规划：In1.Cu = GND 平面、In2.Cu = VLED 平面，两个外层放信号。
DRC 无新增违规（无 copper_edge_clearance / clearance / track_width error）；
八项校验器全绿。
Other:
- copper layers 2 -> 4
Changed lines of the file:
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@@
 	(layers
 		(0 "F.Cu" signal)
-		(31 "B.Cu" signal)
+		(4 "In1.Cu" signal)
+		(6 "In2.Cu" signal)
+		(2 "B.Cu" signal)
 		(9 "F.Adhes" user "F.Adhesive")
 		(11 "B.Adhes" user "B.Adhesive")
 		(13 "F.Paste" user)
 		(15 "B.Paste" user)
-		(5 "F.SilkS" user "F.SilkS")
-		(7 "B.SilkS" user "B.SilkS")
+		(5 "F.SilkS" user)
+		(7 "B.SilkS" user)
 		(1 "F.Mask" user)
 		(3 "B.Mask" user)
