File: hardware/pcb/StarShield/Starshield.kicad_pcb (KiCad board)
At the start: 2 copper layers, 374.7 x 151.1 mm, 321 parts, among them J1 USB_C_Receptacle_USB2.0_16P, J2 B2B-PH-K-S, J3A nice!nano v2 左列 (PM 1-12), J3B nice!nano v2 右列 (PM 13-24), Q1 AO3401A, Q2 2N7002, SW1 Esc, SW10 F7, SW11 F8, SW12 F9, SW13 F10, SW14 F11, SW15 F12, SW16 Delete, SW17 /, SW18 *, SW19 -, SW2 FN, SW20 +, SW21 ~/`, SW22 !/1, SW23 @/2, SW24 #/3, SW25 $/4, SW26 %/5, SW27 ^/6, SW28 &/7, SW29 */8, SW3 Num Lock, SW30 (/9, SW31 )/0, SW32 _/-, SW33 +/=, SW34 Back Space, SW35 Delete, SW36 7/Home, SW37 8/↑, SW38 9/PgUp, SW39 Tab, SW4 F1, SW40 Q, SW41 W, SW42 E, SW43 R, SW44 T, SW45 Y, SW46 U, SW47 I, SW48 O, SW49 P, SW5 F2, SW50 {/[, SW51 }/], SW52 Enter, SW53 4/←, SW54 5, SW55 6/→, SW56 Caps Lock, SW57 A, SW58 S, SW59 D, SW6 F3, SW60 F, SW61 G, SW62 H, SW63 J, SW64 K, SW65 L, SW66 :/;, SW67 "/', SW68 Enter, SW69 1/End, SW7 F4, SW70 2/↓, SW71 3/PgDn, SW72 Shift, SW73 Z, SW74 X, SW75 C, SW76 V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

Commit message: feat(pcb): USB-C 移左上角 / 三档开关移右上角；改为 4 层板
用户 2026-09-19 定的两处摆位：
- J1 (USB-C) 210,5.5 -> 15,5.5（左上角）；**R1/R2（CC 下拉）与 F1 随连接器左移**
  —— CC 走线必须短，否则是 USB-C 坏实践。代价：VBUS 从 F1 到 U1 变成约 230mm 长线
  （0.8mm 宽、1A，电气无碍）。
- SW96（三档模式开关）75,12 -> 360,6（右上角）。代价：MODE0/1/2 三条线从约 35mm
  变成约 320mm（μA 级信号，无碍）。

层数：2 -> **4 层**。⚠️ 关键教训：**层数属设计数据，必须由生成器产出** ——
先前用 MCP add_layer 加的 In1/In2 被下一次 gen_pcb.py 覆盖掉了。现写死进 gen_pcb.py 的
LAYERS，层号与顺序**照抄 KiCad 自己写出的形式**（B.Cu 的 id 是 2 而不是 31；
KiCad 还会去掉 F.SilkS/B.SilkS 的别名串）。

叠层规划：In1.Cu = GND 平面、In2.Cu = VLED 平面，两个外层放信号。
DRC 无新增违规（无 copper_edge_clearance / clearance / track_width error）；
八项校验器全绿。
Parts:
- moved SW96 285.1 mm to (360.0, 6.00)
- moved F1 221.6 mm to (18.5, 12.5)
- moved R1 216.1 mm to (12.0, 12.5)
- moved R2 216.1 mm to (12.0, 16.0)
- moved J1 195.0 mm to (15.0, 5.50)
Other:
- copper layers 2 -> 4
Changed lines of the file:
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@@
 	(layers
 		(0 "F.Cu" signal)
-		(31 "B.Cu" signal)
+		(4 "In1.Cu" signal)
+		(6 "In2.Cu" signal)
+		(2 "B.Cu" signal)
 		(9 "F.Adhes" user "F.Adhesive")
 		(11 "B.Adhes" user "B.Adhesive")
 		(13 "F.Paste" user)
 		(15 "B.Paste" user)
-		(5 "F.SilkS" user "F.SilkS")
-		(7 "B.SilkS" user "B.SilkS")
+		(5 "F.SilkS" user)
+		(7 "B.SilkS" user)
 		(1 "F.Mask" user)
 		(3 "B.Mask" user)
@@
 	(footprint "Fuse:Fuse_1812_4532Metric"
 		(layer "F.Cu")
-		(at 240 6 0)
+		(at 18.5 12.5 0)
 		(version 20260206)
 		(generator "kicad-footprint-generator")
@@
 	(footprint "Connector_USB:USB_C_Receptacle_HRO_TYPE-C-31-M-12"
 		(layer "F.Cu")
-		(at 210 5.5 0)
+		(at 15 5.5 0)
 		(version 20260206)
 		(generator "pcbnew")
@@
 	(footprint "Resistor_SMD:R_0603_1608Metric"
 		(layer "F.Cu")
-		(at 228 6 0)
+		(at 12 12.5 0)
 		(version 20260206)
 		(generator "kicad-footprint-generator")
@@
 	(footprint "Resistor_SMD:R_0603_1608Metric"
 		(layer "F.Cu")
-		(at 228 11 0)
+		(at 12 16 0)
 		(version 20260206)
 		(generator "kicad-footprint-generator")
@@
 	(footprint "Button_Switch_SMD:SW_SP3T_PCM13"
 		(layer "F.Cu")
-		(at 75 12 0)
+		(at 360 6 0)
 		(version 20260206)
 		(generator "pcbnew")

Commit message: fix(pcb): 三档开关按使用体验微调至 (350,11)（原 360,6 太贴角）
用户反馈「太偏了，考虑实际使用体验」⇒ 往左下各挪 10mm / 5mm。
新位置外廓 x 344.1..355.9、y 8.55..14.4：离板右缘 18.8mm、离顶肩下沿 9.6mm、
与 J2 水平间隙 8.0mm，四周均有余量。

同时把封装姿态的实测结论写进 pcb_design.py 注释（读 KiCad 官方 SW_SP3T_PCM13）：
本体 9.7 x 2.55mm 沿 X 长；四个信号脚在 -Y 侧（y=-1.43）；
**操作柄在 +Y 侧伸出**（F.CrtYd 到 y=3.4）⇒ rot=0 时柄指向键区方向；
若希望柄朝键盘后壁，把 rot 改成 180 即可（一行）。

八项校验器全绿；DRC 无新增违规。
Parts:
- moved SW96 11.2 mm to (350.0, 11.0)
Changed lines of the file:
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@@
 	(footprint "Button_Switch_SMD:SW_SP3T_PCM13"
 		(layer "F.Cu")
-		(at 360 6 0)
+		(at 350 11 0)
 		(version 20260206)
 		(generator "pcbnew")

Commit message: feat(pcb): 三档开关按侧壁开口定型（rot=180, y=2.5）并锁定档位物理顺序
用户 2026-09-19 定：「外壳开口开在侧面（和 USB-C 同一面），滑块式，
从左往右依次是 2.4G / 蓝牙 / 有线」。

- **rot 0 -> 180**：柄朝后壁（-Y）。侧壁开口要求柄能穿过外壳侧壁
- **y 11 -> 2.5**：柄尖板坐标 y = y0-3.4 = -0.9 ⇒ **探出板边 0.9mm**，才能伸进侧壁开孔。
  ⚠️ 这与先前「往左下挪」的「下」冲突（侧壁开口物理上要求靠边），按硬约束取舍；
  X 保留用户左移后的 350
- 最小的铜是机械焊盘 y=1.07，仍 >= 板边 0.5mm ✓

档位物理顺序的依据（一手，非推测）：C&K PCM 手册 SP3T 连接表 1-3 / 2-3 / 3-4
⇒ pin3=公共端（接 GND）、POS1->pin1、POS2->pin2、POS3->pin4；
封装焊盘 pin1/2/3/4 沿 X 依次 -3/-1.5/+1.5/+3mm。
**rot=180 镜像 X** ⇒ 板坐标自左向右 = POS3/POS2/POS1 = pin4/pin2/pin1
= MODE2/MODE1/MODE0 = **2.4G / 蓝牙 / 有线** ✓ 正好等于用户要求，原理图无需改动。

⚠️ 改 SW96 的 rot 或改这三条接线都会反转顺序 —— 推算已写进
pcb_design.py 与 starshield.overlay 的注释。

八项校验器全绿；silk_edge_clearance 1->3 条警告属预期（丝印随柄探出板边）。
Parts:
- moved SW96 8.50 mm to (350.0, 2.50), turned to 180 degrees
Changed lines of the file:
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@@
 	(footprint "Button_Switch_SMD:SW_SP3T_PCM13"
 		(layer "F.Cu")
-		(at 350 11 0)
+		(at 350 2.5 180)
 		(version 20260206)
 		(generator "pcbnew")

Commit message: feat(pcb): B4 布线（4 层，信号走外层 + 内层平面/铺铜）—— 99.3% 布通，剩 6 条待收
用 Freerouting 2.4.1（Java 25）自动布线，产物 = 3696 段走线 + 296 个过孔 +
3 个已填充铺铜区（In1.Cu=GND 平面、In2.Cu=VLED 平面、B.Cu=GND）。

关键做法与实测：
- **内层声明为 power 层**（DSN 里 In1.Cu/In2.Cu 的 type 由 signal 改 power）
  ⇒ Freerouting 只用 F.Cu/B.Cu 走信号，内层腾空给平面。
  不加这一步时 4 层跑法反而更差（73 未布且被提前中断）。
- VLED 交给布线器时宽度由 2.0mm 降到 0.25mm（只保连通性），载流靠 In2 平面；
  2.0mm 宽在 19.05mm 键位栅格里连 95 个焊盘会让布线器跑不动（实测 5 分钟一个 pass 都完不成）。
- 收敛轨迹：121 -> 42 -> 20 -> 9 -> 7 -> 6（10 pass / 20 分钟，-mt 4）。

新增 docs/_tools/route_freerouting.py：把「DSN 预处理 + 调宽度 + 调 Freerouting +
摘要」固化成一条命令，含 Java 25 / gh-proxy 镜像 / 线程数等本机坑的说明。

DRC（kicad-cli）与布线相关的 error 全部为 0：
track_width 0、clearance 0、tracks_crossing 0、shorting_items 0。
- 收尾时把 U1 散热扇出区的 24 段短 GND 定为 0.127mm（5mil，1oz 铜工艺下限），
  并把工程文件 min_track_width 由 0.2 调到 0.127 —— 因为加宽到 0.2 会与相邻焊盘
  冲突（实测多出 4 条 clearance，间隙违规比线宽违规更危险）。
  真正修复是把这几颗散热过孔挪进 U1 散热焊盘内（已记入 handoff 待办）。

未完成（投板前必须清零）：剩 6 条未连通 —— VLED 断口、COL0、D17-A x2、VBUS 等。
已试过手工直线补线，会穿过其余走线（实测 5 处 tracks_crossing + 1 处 shorting_items），
已全部撤销；剩余部分需要用 KiCad GUI 或更谨慎的分段走线处理。

校验器同步修正：
- verify_pcb.py 的 VLED 断言改为**读工程文件**的 net_settings.classes
  —— KiCad 8+ 保存时会把网络类从板文件挪到 .kicad_pro，旧口径会假失败。
- DRC_ALLOW 的 unconnected_items 理由更新为「布线未完成，剩 6 条」。
八项校验器全绿。
Routing:
- net GND: track 0.00 -> 2550.3 mm, vias 0 -> 18
- net VLED: track 0.00 -> 2109.7 mm, vias 0 -> 2
- net ROW4: track 0.00 -> 709.2 mm, vias 0 -> 1
- net ROW2: track 0.00 -> 687.0 mm, vias 0 -> 4
- net ROW1: track 0.00 -> 639.2 mm, vias 0 -> 5
- net ROW0: track 0.00 -> 632.5 mm, vias 0 -> 6
- net ROW5: track 0.00 -> 630.8 mm, vias 0 -> 3
- net ROW3: track 0.00 -> 622.2 mm, vias 0 -> 6
- net COL10: track 0.00 -> 419.3 mm, vias 0 -> 7
- net COL9: track 0.00 -> 395.6 mm, vias 0 -> 8
- net COL7: track 0.00 -> 392.7 mm, vias 0 -> 7
- net RGB（95 颗 SK6812MINI-E 数据链）/LED_DIN_17: track 0.00 -> 371.3 mm, vias 0 -> 2
- net COL15: track 0.00 -> 370.8 mm, vias 0 -> 6
- net RGB（95 颗 SK6812MINI-E 数据链）/LED_DIN_35: track 0.00 -> 361.7 mm, vias 0 -> 4
- net COL8: track 0.00 -> 358.4 mm, vias 0 -> 7
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- added copper zone on B.Cu, net GND
- added copper zone on In1.Cu, net GND
- added copper zone on In2.Cu, net VLED
Other:
- net class Default removed
- net class Power removed
- net class VLED removed
