File: hardware/pcb/StarShield/Starshield.kicad_pcb (KiCad board)
At the start: 4 copper layers, 374.7 x 151.1 mm, 321 parts, among them J1 USB_C_Receptacle_USB2.0_16P, J2 B2B-PH-K-S, J3A nice!nano v2 左列 (PM 1-12), J3B nice!nano v2 右列 (PM 13-24), Q1 AO3401A, Q2 2N7002, SW1 Esc, SW10 F7, SW11 F8, SW12 F9, SW13 F10, SW14 F11, SW15 F12, SW16 Delete, SW17 /, SW18 *, SW19 -, SW2 FN, SW20 +, SW21 ~/`, SW22 !/1, SW23 @/2, SW24 #/3, SW25 $/4, SW26 %/5, SW27 ^/6, SW28 &/7, SW29 */8, SW3 Num Lock, SW30 (/9, SW31 )/0, SW32 _/-, SW33 +/=, SW34 Back Space, SW35 Delete, SW36 7/Home, SW37 8/↑, SW38 9/PgUp, SW39 Tab, SW4 F1, SW40 Q, SW41 W, SW42 E, SW43 R, SW44 T, SW45 Y, SW46 U, SW47 I, SW48 O, SW49 P, SW5 F2, SW50 {/[, SW51 }/], SW52 Enter, SW53 4/←, SW54 5, SW55 6/→, SW56 Caps Lock, SW57 A, SW58 S, SW59 D, SW6 F3, SW60 F, SW61 G, SW62 H, SW63 J, SW64 K, SW65 L, SW66 :/;, SW67 "/', SW68 Enter, SW69 1/End, SW7 F4, SW70 2/↓, SW71 3/PgDn, SW72 Shift, SW73 Z, SW74 X, SW75 C, SW76 V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

Commit message: feat(pcb): 给 VLED 补 43 个过孔，In2 平面成为真正的 2.4A 配电层；未连通 6 -> 5
问题：布线后 VLED 只有 2 个过孔（都在板子右侧），2.4A 仍主要靠布线器留下的
0.25mm 细走线承载 —— ADR-0007 的载流要求没落地。

做法：新增 add_vled_vias.py ——
候选点取现有 VLED F.Cu 走线的中点（保证落在自己的铜上），按 22mm 抽稀，
再对其它网络的焊盘/走线/过孔与 NPTH 做间距预筛，通过的写成
(via size 0.6 drill 0.3 layers F.Cu-B.Cu net VLED)。
放入 55 个后 DRC 报出 23 处冲突（预筛漏了 B.Cu 上的热插拔座焊盘：
自画封装同一引脚号有 PTH + B.Cu SMD 两个焊盘，解析器按引脚号取值时丢了其一）
⇒ 再用 drop_bad_vias.py 按 DRC 报告删掉被点名的 14 个
⇒ 最终保留 41 个新过孔（VLED 共 43 个），DRC clearance/shorting/track_width 全为 0。

附带收益：**未连通 6 -> 5** —— VLED 那个 24.6mm 断口被 In2 平面本身接通了
（两端各有过孔落到平面上），这也反证了平面确实在导电。

⚠️ 踩到的两个工具坑（都已记入 handoff）：
1. 铺铜的填充多边形是「加过孔之前」算的 ⇒ 新过孔与 B.Cu 的 GND 铺铜重叠，
   DRC 一次性报出 216 条 clearance/hole_clearance；**重填铺铜后降到 18 条**。
   所以「改完板子必须重填铺铜」。
2. MCP 的 **open_board 对同一路径不会重新读盘**，此时 save_board 会用陈旧的
   内存内容覆盖磁盘（本轮丢过一次 55 个过孔 + 线宽改动）；
   正确做法是用 **reload_board**，而且 MCP 的 save_board 还会把 .kicad_pro 的
   min_track_width 一起写回旧值 —— 改完脚本后不要再调 MCP 的保存类工具。

八项校验器全绿；剩 5 条未连通（COL0 / D17-A x2 / VBUS / 另 1）待收。
Routing:
- net VLED: vias 2 -> 43
