File: hardware/pcb/StarShield/Starshield.kicad_pcb (KiCad board)
At the start: 4 copper layers, 374.7 x 151.1 mm, 321 parts, among them J1 USB_C_Receptacle_USB2.0_16P, J2 B2B-PH-K-S, J3A nice!nano v2 左列 (孔 1-13), J3B nice!nano v2 右列 (孔 1-13), Q1 AO3401A, Q2 2N7002, SW1 Esc, SW10 F7, SW11 F8, SW12 F9, SW13 F10, SW14 F11, SW15 F12, SW16 Delete, SW17 /, SW18 *, SW19 -, SW2 FN, SW20 +, SW21 ~/`, SW22 !/1, SW23 @/2, SW24 #/3, SW25 $/4, SW26 %/5, SW27 ^/6, SW28 &/7, SW29 */8, SW3 Num Lock, SW30 (/9, SW31 )/0, SW32 _/-, SW33 +/=, SW34 Back Space, SW35 Delete, SW36 7/Home, SW37 8/↑, SW38 9/PgUp, SW39 Tab, SW4 F1, SW40 Q, SW41 W, SW42 E, SW43 R, SW44 T, SW45 Y, SW46 U, SW47 I, SW48 O, SW49 P, SW5 F2, SW50 {/[, SW51 }/], SW52 Enter, SW53 4/←, SW54 5, SW55 6/→, SW56 Caps Lock, SW57 A, SW58 S, SW59 D, SW6 F3, SW60 F, SW61 G, SW62 H, SW63 J, SW64 K, SW65 L, SW66 :/;, SW67 "/', SW68 Enter, SW69 1/End, SW7 F4, SW70 2/↓, SW71 3/PgDn, SW72 Shift, SW73 Z, SW74 X, SW75 C, SW76 V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

Commit message: feat(power): 方案①落地 —— 模块 B+/RAW 由 OUT 改接 VBAT（插模块口即充电）；模块整组左移 + J1 让位
背景（用户质疑成立）：商业键盘一律「一个口 = 数据 + 充电」（Kisnt KN85 / 雷柏 V700-8A /
CHERRY KW 9200 官方口径）；社区 nice!nano 方案把电池挂在模块自带充电器输出上，插模块口即充电。
我们原先把电池接自研 BQ24072 的 BAT、模块挂 OUT ⇒ 模块充电器的电流进不了电池
（OUT→BAT 不是充电路径）⇒ 有线模式下充不上电。

改动：
- 电路：J3B 孔1/孔2（B+/RAW）网络 OUT -> VBAT；VBAT 由电源子图局部网升为跨子图全局网
  （power_design.py 与 control_design.py 的 GLOBAL_NETS 各加 VBAT）
- 子图：power.kicad_sch / control.kicad_sch 重生成（版式自检通过）
- 校验：verify_control 断言改为「VBAT 跨图连通（J3B 孔1/2 + U1/J2/C3）」+
  「OUT 不再挂 J3B」；网表类五项校验全绿
- 几何（B6-2）：nice!nano 插座整组左移 30.46 mm（孔1 x=7.00、口面 x=1.70 与壳面齐平）；
  J1/R1/R2/F1 让位到 x=155-168；pcb_design.py 同步
- 板文件：J3B 孔1/2 改网为 VBAT（旧 OUT 走线已随左移一并清除）
- 文档：power-architecture.md §1 / bq24072-pinout.md §2.3 / decisions.md 电源段各加「重载仍接 OUT、
  模块为唯一例外」的修订说明；量测文档 §6.6 记录完整对标与代价

⚠️ 遗留（下一步）：肩部走线缺口待补（左移时删了 76 项），Freerouting 正在用新网表全板重布；
完成后需重跑 DRC + 七项校验器。
Parts:
- moved F1 149.5 mm to (168.0, 12.0)
- moved R2 147.0 mm to (159.0, 14.0)
- moved J1 145.0 mm to (160.0, 5.50)
- moved R1 143.0 mm to (155.0, 14.0)
- moved J3A 30.5 mm to (9.54, 4.38)
- moved J3B 30.5 mm to (9.54, 19.6)
Connections:
- J3B pad 1: OUT -> 电源 / 充电 / RGB 门控/VBAT
- J3B pad 2: OUT -> 电源 / 充电 / RGB 门控/VBAT
Routing:
- net GND: track 2550.3 -> 2469.8 mm
- net OUT: track 298.5 -> 276.9 mm
- net 电源 / 充电 / RGB 门控/VCHG_IN: track 243.9 -> 222.4 mm
- net 电源 / 充电 / RGB 门控/CC2: track 18.6 -> 0.00 mm, vias 2 -> 0
- net VBUS: track 18.3 -> 0.00 mm, vias 3 -> 0
- net VCC: track 147.5 -> 131.3 mm
- net 电源 / 充电 / RGB 门控/CC1: track 13.6 -> 0.00 mm, vias 2 -> 0
- net 控制板 / MCU / 595 / 模式开关/MODE2: track 306.7 -> 293.9 mm
- net LED_DIN: track 51.6 -> 43.2 mm
- net 控制板 / MCU / 595 / 模式开关/595_MOSI: track 44.0 -> 35.8 mm
- net 控制板 / MCU / 595 / 模式开关/595_RCLK: track 82.3 -> 75.1 mm
- net 控制板 / MCU / 595 / 模式开关/595_SCK: track 79.3 -> 73.1 mm
- net ROW4: track 709.2 -> 703.8 mm
- net 控制板 / MCU / 595 / 模式开关/MODE1: track 298.7 -> 293.7 mm
- net RGB_PWR_EN: track 236.2 -> 231.7 mm
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
Commit message: refactor(pcb): 左侧接口簇定稿 —— 模块下移 5.78mm 让出左上角；充电口回左上角(x=15)、开关紧邻(x=33)、模块口留左壁(y=17.8)
用户定稿排布：模块口在左侧壁、充电口在左上角、开关放充电口旁边。空间核算见 docs/nice-nano-physical-verification.md §6.7：左侧壁键区前仅 ~30mm 可用，三者需挤在 y 0-8 ⇒ 模块下移至两排 y=10.16/25.40（距键区仍有 3.8mm）。板框仍 374.71x151.06，未加高额头。pcb_design.py 已同步；板/定位板由 gen_pcb.py 重新生成（布线待重做）。
Parts:
- moved SW96 317.0 mm to (33.0, 2.50)
- moved J1 145.0 mm to (15.0, 5.50)
- moved R1 143.0 mm to (12.0, 14.0)
- moved R2 143.0 mm to (16.0, 14.0)
- moved F1 142.0 mm to (26.0, 14.0)
- moved J3A 5.78 mm to (9.54, 10.2)
- moved J3B 5.78 mm to (9.54, 25.4)
Connections:
- net 电源 / 充电 / RGB 门控/VBAT renamed VBAT
Routing:
- net GND: track 2469.8 -> 0.00 mm, vias 18 -> 0
- net VLED: track 2109.7 -> 0.00 mm, vias 43 -> 0
- net ROW4: track 703.8 -> 0.00 mm, vias 1 -> 0
- net ROW2: track 686.4 -> 0.00 mm, vias 4 -> 0
- net ROW1: track 637.4 -> 0.00 mm, vias 5 -> 0
- net ROW0: track 630.8 -> 0.00 mm, vias 6 -> 0
- net ROW5: track 628.2 -> 0.00 mm, vias 3 -> 0
- net ROW3: track 620.3 -> 0.00 mm, vias 6 -> 0
- net COL10: track 419.3 -> 0.00 mm, vias 7 -> 0
- net COL9: track 395.6 -> 0.00 mm, vias 8 -> 0
- net COL7: track 392.7 -> 0.00 mm, vias 7 -> 0
- net RGB（95 颗 SK6812MINI-E 数据链）/LED_DIN_17: track 371.3 -> 0.00 mm, vias 2 -> 0
- net COL15: track 370.8 -> 0.00 mm, vias 6 -> 0
- net RGB（95 颗 SK6812MINI-E 数据链）/LED_DIN_35: track 361.7 -> 0.00 mm, vias 4 -> 0
- net COL8: track 358.4 -> 0.00 mm, vias 7 -> 0
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- removed copper zone on B.Cu, net GND
- removed copper zone on In1.Cu, net GND
- removed copper zone on In2.Cu, net VLED
Other:
- net class Default added: clearance 0.2, trace_width 0.25, via_dia 0.6, via_drill 0.3
- net class Power added: clearance 0.2, trace_width 0.8, via_dia 0.8, via_drill 0.4
- net class VLED added: clearance 0.25, trace_width 2.0, via_dia 1.2, via_drill 0.6
